File: rf-synth.kicad_sch (KiCad schematic)
At the start: 66 parts, among them J1 SMA-F, J2 SMA-F, J3 SMA-F, J4 SMA-F, U1 LMX2594, U2 AP7361C-33E, U3 RP2040_XIAO, Y1 ASCO

Commit message: routed more
Parts:
- U1: footprint Package_DFN_QFN:VQFN-40-1EP_6x6mm_P0.5mm_EP3.5x3.5mm_ThermalVias -> Package_DFN_QFN:VQFN-40-1EP_6x6mm_P0.5mm_EP3.5x3.5mm
Changed lines of the file:
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@@
 			)
 		)
-		(property "Footprint" "Package_DFN_QFN:VQFN-40-1EP_6x6mm_P0.5mm_EP3.5x3.5mm_ThermalVias"
+		(property "Footprint" "Package_DFN_QFN:VQFN-40-1EP_6x6mm_P0.5mm_EP3.5x3.5mm"
 			(at 273.05 176.53 0)
 			(effects
