File: rf-synth.kicad_pcb (KiCad board)
At the start: 4 copper layers, 50 x 50 mm, 66 parts, among them J1 SMA-F, J2 SMA-F, J3 SMA-F, J4 SMA-F, U1 LMX2594, U2 AP7361C-33E, U3 RP2040_XIAO, Y1 ASCO

Commit message: routed some
Parts:
- moved C7 2.15 mm to (165.5, 114.0)
- moved C3 1.58 mm to (165.2, 111.2)
- moved C6 1.56 mm to (155.8, 122.0), turned to -90 degrees
- moved C10 1.35 mm to (163.8, 109.8)
- moved C12 0.79 mm to (162.0, 108.2)
- moved FB3 0.70 mm to (155.0, 124.7)
- moved C27 0.50 mm to (159.8, 128.0)
- moved J2 0.22 mm to (181.3, 122.0)
- moved J1 0.21 mm to (181.3, 113.0)
Routing:
- net /SYSREFREQ: track 0.00 -> 39.0 mm, vias 0 -> 2
- net /RAMPCLK: track 0.00 -> 34.1 mm, vias 0 -> 2
- net /RAMPDIR: track 0.00 -> 29.8 mm, vias 0 -> 2
- net /SYNC: track 0.00 -> 25.2 mm, vias 0 -> 2
- net /ENABLE: track 0.00 -> 21.8 mm, vias 0 -> 2
- net /VTUNE: track 0.00 -> 21.5 mm, vias 0 -> 2
- net /CPOUT: track 0.00 -> 20.5 mm
- net Net-(Y1-OUT): track 0.00 -> 13.6 mm, vias 0 -> 2
- net Net-(J1-In): track 0.00 -> 11.3 mm
- net Net-(J2-In): track 0.00 -> 11.3 mm
- net Net-(U1-VccVCO2): track 0.00 -> 9.10 mm
- net Net-(J4-In): track 0.00 -> 8.93 mm
- net Net-(J3-In): track 0.00 -> 8.84 mm
- net Net-(U1-VccDIG): track 0.00 -> 8.13 mm
- net Net-(U1-RFoutAP): track 0.00 -> 7.41 mm
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
Commit message: routed more
Parts:
- U1: footprint Package_DFN_QFN:VQFN-40-1EP_6x6mm_P0.5mm_EP3.5x3.5mm_ThermalVias -> Package_DFN_QFN:VQFN-40-1EP_6x6mm_P0.5mm_EP3.5x3.5mm
- moved J4 2.08 mm to (153.0, 135.4)
- moved J2 2.03 mm to (181.2, 124.0)
- moved J1 1.97 mm to (181.2, 111.0)
- moved J3 1.75 mm to (166.0, 135.4)
- moved C13 0.60 mm to (163.5, 120.6)
- moved C14 0.60 mm to (163.5, 121.6)
- moved C11 0.25 mm to (150.2, 112.8)
- moved FB6 0.15 mm to (165.2, 122.9)
Routing:
- net /SCK: track 2.28 -> 50.2 mm, vias 1 -> 2
- net /MOSI: track 2.83 -> 44.6 mm, vias 1 -> 2
- net /MUXOUT: track 0.00 -> 31.3 mm, vias 0 -> 2
- net /CS: track 0.00 -> 19.3 mm, vias 0 -> 2
- net +3V3: track 0.00 -> 17.3 mm, vias 0 -> 19
- net +5V: track 0.00 -> 10.4 mm
- net GND: track 0.00 -> 6.35 mm, vias 0 -> 384
- net VCCRF: track 1.73 -> 7.91 mm, vias 0 -> 10
- net Net-(J1-In): track 11.3 -> 16.9 mm
- net Net-(J2-In): track 11.3 -> 16.7 mm
- net Net-(J4-In): track 8.93 -> 14.0 mm
- net Net-(J3-In): track 8.84 -> 13.9 mm
- net Net-(U1-VccMASH): track 2.16 -> 6.84 mm
- net Net-(U1-VccCP): track 4.91 -> 7.21 mm
- net Net-(Y1-OUT): track 13.6 -> 15.6 mm
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- added copper zone on In2.Cu, net +3V3
- added copper zone on B.Cu, net GND
- added copper zone on F.Cu, net GND
- added copper zone on In1.Cu, net GND
- added copper zone on In2.Cu, net VCCRF

Commit message: maybe fucked
Parts:
- moved J4 0.28 mm to (153.2, 135.4)
- moved J3 0.25 mm to (166.2, 135.4)
Routing:
- net Net-(J1-In): track 16.9 -> 13.5 mm
- net Net-(J4-In): track 14.0 -> 10.8 mm
- net Net-(J2-In): track 16.7 -> 13.6 mm
- net Net-(J3-In): track 13.9 -> 10.8 mm
- net GND: vias 384 -> 385
Changed lines of the file:
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@@
 	(footprint "0thaumati-footprintslib:ADAMTECH_RF2-143-T-17-50-G"
 		(layer "F.Cu")
-		(at 152.96825 135.4127)
+		(at 153.25 135.4127)
 		(property "Reference" "J4"
 			(at -0.325 -6.635 0)
@@
 	(footprint "0thaumati-footprintslib:ADAMTECH_RF2-143-T-17-50-G"
 		(layer "F.Cu")
-		(at 166 135.4127)
+		(at 166.25 135.4127)
 		(property "Reference" "J3"
 			(at -0.325 -6.635 0)
@@
 	)
 	(via
-		(at 131.8 107.7)
+		(at 132.2 107.9)
 		(size 0.6)
 		(drill 0.3)
@@
 	)
 	(via
-		(at 178.7 134.7)
+		(at 179.4 134.4)
 		(size 0.6)
 		(drill 0.3)
@@
 	)
 	(via
-		(at 131.7 102)
+		(at 132.3 102.5)
 		(size 0.6)
 		(drill 0.3)
@@
 	)
 	(via
-		(at 131.6 97.5)
+		(at 132.2 97.5)
 		(size 0.6)
 		(drill 0.3)
@@
 	)
 	(via
+		(at 155.9 97.6)
+		(size 0.6)
+		(drill 0.3)
+		(layers "F.Cu" "B.Cu")
+		(free yes)
+		(net 1)
+	)
+	(via
 		(at 143.1 125.2)
 		(size 0.6)
@@
 	)
 	(via
-		(at 132 100)
+		(at 132.3 99.9)
 		(size 0.6)
 		(drill 0.3)
@@
 	)
 	(via
-		(at 162.75 129.75)
+		(at 162.3 129.7)
 		(size 0.6)
 		(drill 0.3)
@@
 	)
 	(segment
-		(start 171.75 115.5)
-		(end 176.21825 111.03175)
+		(start 173.070426 114.179574)
+		(end 175.225286 112.024714)
 		(width 0.35)
 		(layer "F.Cu")
@@
 	(segment
 		(start 168.9425 115.5)
-		(end 171.75 115.5)
+		(end 169.882637 115.5)
 		(width 0.35)
 		(layer "F.Cu")
@@
 	)
 	(segment
-		(start 176.21825 111.03175)
-		(end 179.2502 111.03175)
+		(start 177.622512 111.03175)
+		(end 180.96825 111.03175)
 		(width 0.35)
 		(layer "F.Cu")
 		(net 26)
 	)
-	(segment
-		(start 176.21825 111.03175)
-		(end 180.96825 111.03175)
+	(arc
+		(start 169.882637 115.5)
+		(mid 171.607856 115.156833)
+		(end 173.070426 114.179574)
+		(width 0.35)
+		(layer "F.Cu")
+		(net 26)
+	)
+	(arc
+		(start 177.622512 111.03175)
+		(mid 176.325142 111.289813)
+		(end 175.225286 112.024714)
 		(width 0.35)
 		(layer "F.Cu")
@@
 	(segment
 		(start 162.6 117.15)
-		(end 164 115.75)
+		(end 163.121321 116.628679)
 		(width 0.35)
 		(layer "F.Cu")
@@
 	)
 	(segment
-		(start 164 115.75)
+		(start 165.242641 115.75)
 		(end 166.75 115.75)
 		(width 0.35)
@@
 		(net 27)
 	)
+	(arc
+		(start 165.242641 115.75)
+		(mid 164.094591 115.978361)
+		(end 163.121321 116.628679)
+		(width 0.35)
+		(layer "F.Cu")
+		(net 27)
+	)
 	(segment
 		(start 168.9425 119.5)
-		(end 171.46825 119.5)
+		(end 169.766622 119.5)
 		(width 0.35)
 		(layer "F.Cu")
@@
 	)
 	(segment
-		(start 171.46825 119.5)
-		(end 176 124.03175)
+		(start 172.671482 120.703232)
+		(end 175.125638 123.157388)
 		(width 0.35)
 		(layer "F.Cu")
@@
 	)
 	(segment
-		(start 176.5 124.03175)
-		(end 179.25 124.03175)
+		(start 177.236535 124.03175)
+		(end 181 124.03175)
 		(width 0.35)
 		(layer "F.Cu")
 		(net 28)
 	)
-	(segment
-		(start 176.5 124.03175)
-		(end 181 124.03175)
+	(arc
+		(start 175.125638 123.157388)
+		(mid 176.094126 123.804511)
+		(end 177.236535 124.03175)
 		(width 0.35)
 		(layer "F.Cu")
 		(net 28)
 	)
-	(segment
-		(start 176 124.03175)
-		(end 176.5 124.03175)
+	(arc
+		(start 172.671482 120.703232)
+		(mid 171.338721 119.81271)
+		(end 169.766622 119.5)
 		(width 0.35)
 		(layer "F.Cu")
@@
 	(segment
 		(start 162.5875 117.8375)
-		(end 163.945 119.195)
+		(end 163.066321 118.316321)
 		(width 0.35)
 		(layer "F.Cu")
@@
 	)
 	(segment
-		(start 163.945 119.195)
+		(start 165.187641 119.195)
 		(end 166.75 119.195)
 		(width 0.35)
@@
 		(net 29)
 	)
+	(arc
+		(start 163.066321 118.316321)
+		(mid 164.039591 118.966639)
+		(end 165.187641 119.195)
+		(width 0.35)
+		(layer "F.Cu")
+		(net 29)
+	)
 	(segment
 		(start 160.2775 123.5)
@@
 	)
 	(segment
-		(start 166 130.5)
-		(end 166 130.9)
+		(start 162.285603 126.985603)
+		(end 165.632373 130.332373)
 		(width 0.35)
 		(layer "F.Cu")
@@
 	)
 	(segment
-		(start 161.75 125.6925)
-		(end 161.75 126.25)
+		(start 166.25 131.823457)
+		(end 166.25 134.824)
 		(width 0.35)
 		(layer "F.Cu")
 		(net 31)
 	)
-	(segment
-		(start 161.75 126.25)
-		(end 166 130.5)
+	(arc
+		(start 165.632373 130.332373)
+		(mid 166.089484 131.016488)
+		(end 166.25 131.823457)
 		(width 0.35)
 		(layer "F.Cu")
 		(net 31)
 	)
-	(segment
-		(start 166 130.9)
-		(end 166 135.2)
-		(width 0.35)
-		(layer "F.Cu")
-		(net 31)
-	)
-	(segment
-		(start 166 130.9)
-		(end 166 133.4934)
+	(arc
+		(start 161.75 125.6925)
+		(mid 161.889199 126.392341)
+		(end 162.285603 126.985603)
 		(width 0.35)
 		(layer "F.Cu")
@@
 	)
 	(segment
-		(start 161.4725 122.7225)
-		(end 160.85 122.1)
+		(start 161.179607 122.429607)
+		(end 161.142893 122.392893)
 		(width 0.35)
 		(layer "F.Cu")
@@
 	(segment
 		(start 161.4725 123.5)
-		(end 161.4725 122.7225)
+		(end 161.4725 123.136714)
 		(width 0.35)
 		(layer "F.Cu")
@@
 	)
 	(segment
-		(start 160.85 122.1)
-		(end 160.85 120.75)
+		(start 160.85 121.685786)
+		(end 160.85 121.164214)
 		(width 0.35)
 		(layer "F.Cu")
@@
 	)
 	(segment
-		(start 160.85 120.75)
+		(start 160.557107 120.457107)
 		(end 160 119.9)
 		(width 0.35)
@@
 		(net 32)
 	)
+	(arc
+		(start 161.179607 122.429607)
+		(mid 161.39638 122.75403)
+		(end 161.4725 123.136714)
+		(width 0.35)
+		(layer "F.Cu")
+		(net 32)
+	)
+	(arc
+		(start 161.142893 122.392893)
+		(mid 160.92612 122.06847)
+		(end 160.85 121.685786)
+		(width 0.35)
+		(layer "F.Cu")
+		(net 32)
+	)
+	(arc
+		(start 160.557107 120.457107)
+		(mid 160.77388 120.78153)
+		(end 160.85 121.164214)
+		(width 0.35)
+		(layer "F.Cu")
+		(net 32)
+	)
 	(segment
-		(start 152.96825 131.03175)
-		(end 152.96825 135.2)
+		(start 157.214378 126.985622)
+		(end 153.879237 130.320763)
 		(width 0.35)
 		(layer "F.Cu")
@@
 	)
 	(segment
-		(start 157.75 126.25)
-		(end 152.96825 131.03175)
+		(start 153.25 131.839876)
+		(end 153.25 134.824)
 		(width 0.35)
 		(layer "F.Cu")
 		(net 33)
 	)
-	(segment
-		(start 152.96825 131.03175)
-		(end 152.96825 133.5002)
+	(arc
+		(start 153.879237 130.320763)
+		(mid 153.413533 131.017738)
+		(end 153.25 131.839876)
 		(width 0.35)
 		(layer "F.Cu")
 		(net 33)
 	)
-	(segment
-		(start 157.75 125.6925)
-		(end 157.75 126.25)
+	(arc
+		(start 157.214378 126.985622)
+		(mid 157.610797 126.392338)
+		(end 157.75 125.6925)
 		(width 0.35)
 		(layer "F.Cu")
@@
 	(segment
 		(start 159.4 119.9)
-		(end 158.65 120.65)
+		(end 158.942893 120.357107)
 		(width 0.35)
 		(layer "F.Cu")
@@
 	)
 	(segment
-		(start 158.0275 122.7725)
+		(start 158.0275 123.186714)
 		(end 158.0275 123.5)
 		(width 0.35)
@@
 	)
 	(segment
-		(start 158.65 120.65)
-		(end 158.65 122.15)
+		(start 158.65 121.064214)
+		(end 158.65 121.735786)
 		(width 0.35)
 		(layer "F.Cu")
@@
 	)
 	(segment
-		(start 158.65 122.15)
-		(end 158.0275 122.7725)
+		(start 158.357107 122.442893)
+		(end 158.320393 122.479607)
 		(width 0.35)
 		(layer "F.Cu")
@@
 		(layer "F.Cu")
 		(net 34)
+	)
+	(arc
+		(start 158.357107 122.442893)
+		(mid 158.57388 122.11847)
+		(end 158.65 121.735786)
+		(width 0.35)
+		(layer "F.Cu")
+		(net 34)
+	)
+	(arc
+		(start 158.942893 120.357107)
+		(mid 158.72612 120.68153)
+		(end 158.65 121.064214)
+		(width 0.35)
+		(layer "F.Cu")
+		(net 34)
+	)
+	(arc
+		(start 158.0275 123.186714)
+		(mid 158.10362 122.804031)
+		(end 158.320393 122.479607)
+		(width 0.35)
+		(layer "F.Cu")
+		(net 34)

Commit message: finished board mostly
Routing:
- net GND: vias 385 -> 382
Other:
- board text added: "LMX2594 Test Board"
- board text added: "MX 2025"
- board text added: "RF1"
- board text added: "RF2"
Changed lines of the file:
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@@
 		(tags "capacitor handsolder")
 		(property "Reference" "C24"
-			(at 0 -1.16 0)
+			(at -1.025 -1.1 0)
 			(layer "F.SilkS")
 			(effects
@@
 		(at 136.75 117.75 90)
 		(property "Reference" "Y1"
-			(at 1.31 -2.25 90)
+			(at -1.95 0.75 180)
 			(layer "F.SilkS")
 			(effects
@@
 		(tags "resistor handsolder")
 		(property "Reference" "R6"
-			(at 0 -1.17 90)
+			(at -1.2475 1.35 180)
 			(layer "F.SilkS")
 			(effects
@@
 		(tags "capacitor handsolder")
 		(property "Reference" "C30"
-			(at 0 -1.16 90)
+			(at -0.275 -1.15 90)
 			(layer "F.SilkS")
 			(effects
@@
 		(tags "resistor handsolder")
 		(property "Reference" "R8"
-			(at 0 -1.17 0)
+			(at -1.625 0.6 0)
 			(layer "F.SilkS")
 			(effects
@@
 		(tags "capacitor handsolder")
 		(property "Reference" "C33"
-			(at 0 -1.43 90)
+			(at 0 2.25 180)
 			(layer "F.SilkS")
 			(effects
@@
 		(tags "capacitor handsolder")
 		(property "Reference" "C12"
-			(at 0 -1.43 90)
+			(at 3.15 0 90)
 			(layer "F.SilkS")
 			(effects
@@
 		(tags "capacitor handsolder")
 		(property "Reference" "C10"
-			(at 0 -1.43 90)
+			(at 3.15 0.05 90)
 			(layer "F.SilkS")
 			(effects
@@
 		(tags "capacitor handsolder")
 		(property "Reference" "C13"
-			(at 0 -1.16 0)
+			(at -0.1 -1.4 0)
 			(layer "F.SilkS")
 			(effects
@@
 		(tags "capacitor handsolder")
 		(property "Reference" "C35"
-			(at 0 -1.16 90)
+			(at 2.5325 -0.05 90)
 			(layer "F.SilkS")
 			(effects
@@
 		(tags "resistor handsolder")
 		(property "Reference" "R9"
-			(at 0 -1.17 0)
+			(at 0.212562 1.1 0)
 			(layer "F.SilkS")
 			(effects
@@
 		(tags "capacitor handsolder")
 		(property "Reference" "C11"
-			(at 0 -1.43 0)
+			(at 0 1.45 0)
 			(layer "F.SilkS")
 			(effects
@@
 		(tags "capacitor handsolder")
 		(property "Reference" "C15"
-			(at 0 -1.16 0)
+			(at 2.55 -0.15 0)
 			(layer "F.SilkS")
 			(effects
@@
 		(tags "capacitor handsolder")
 		(property "Reference" "C26"
-			(at 0 -1.16 90)
+			(at 2.65 -0.05 90)
 			(layer "F.SilkS")
 			(effects
@@
 		(tags "capacitor handsolder")
 		(property "Reference" "C27"
-			(at 0 -1.16 90)
+			(at 2.6 -0.05 90)
 			(layer "F.SilkS")
 			(effects
@@
 		(tags "test point SMD pad rectangle square")
 		(property "Reference" "TP3"
-			(at 0 -1.448 0)
+			(at 2.25 -0.25 0)
 			(layer "F.SilkS")
 			(effects
@@
 		)
 		(fp_text user "${REFERENCE}"
-			(at 0 -1.45 0)
+			(at 2.25 -0.25 0)
 			(layer "F.Fab")
 			(effects
@@
 		(tags "capacitor handsolder")
 		(property "Reference" "C8"
-			(at 0 -1.16 90)
+			(at 0.1 1.25 90)
 			(layer "F.SilkS")
 			(effects
@@
 		(tags "capacitor handsolder")
 		(property "Reference" "C7"
-			(at 0 -1.16 0)
+			(at -1.6 0.31 90)
 			(layer "F.SilkS")
 			(effects
@@
 		(tags "capacitor handsolder")
 		(property "Reference" "C16"
-			(at 0 -1.16 0)
+			(at 2.55 0.15 0)
 			(layer "F.SilkS")
 			(effects
@@
 		(tags "resistor handsolder")
 		(property "Reference" "R7"
-			(at 0 -1.17 90)
+			(at 0.6025 0.95 90)
 			(layer "F.SilkS")
 			(effects
@@
 		(tags "capacitor handsolder")
 		(property "Reference" "C20"
-			(at 0 -1.43 90)
+			(at 1.3875 2.25 180)
 			(layer "F.SilkS")
 			(effects
@@
 		(tags "resistor handsolder")
 		(property "Reference" "R3"
-			(at 0 -1.43 90)
+			(at 0 1.4625 90)
 			(layer "F.SilkS")
 			(effects
@@
 		(tags "capacitor handsolder")
 		(property "Reference" "C9"
-			(at 0 -1.43 90)
+			(at 2.75 0.25 90)
 			(layer "F.SilkS")
 			(effects
@@
 		(tags "resistor handsolder")
 		(property "Reference" "R2"
-			(at 0 -1.17 0)
+			(at 1.35 -1.35 0)
 			(layer "F.SilkS")
 			(effects
@@
 		(tags "capacitor handsolder")
 		(property "Reference" "C18"
-			(at 0 -1.43 90)
+			(at 0 -1.5 270)
 			(layer "F.SilkS")
 			(effects
@@
 		(at 181.2127 111.03175 90)
 		(property "Reference" "J1"
-			(at -0.325 -6.635 90)
+			(at 5.03175 -2.7127 90)
 			(layer "F.SilkS")
 			(effects
@@
 		(tags "resistor handsolder")
 		(property "Reference" "R1"
-			(at 0 -1.17 90)
+			(at 0.3 -1.25 90)
 			(layer "F.SilkS")
 			(effects
@@
 		(tags "capacitor handsolder")
 		(property "Reference" "C19"
-			(at 0 -1.43 90)
+			(at -3.3625 0.25 90)
 			(layer "F.SilkS")
 			(effects
@@
 		(at 153.25 135.4127)
 		(property "Reference" "J4"
-			(at -0.325 -6.635 0)
+			(at -5.45 -1.9127 0)
 			(layer "F.SilkS")
 			(effects
@@
 		(tags "capacitor handsolder")
 		(property "Reference" "C14"
-			(at 0 -1.16 0)
+			(at 2.5 -0.1 0)
 			(layer "F.SilkS")
 			(effects
@@
 		(at 181.2127 124.03175 90)
 		(property "Reference" "J2"
-			(at -0.325 -6.635 90)
+			(at -5.76825 -1.9127 90)
 			(layer "F.SilkS")
 			(effects
@@
 		(tags "inductor handsolder")
 		(property "Reference" "FB2"
-			(at 0 -1.43 90)
+			(at 2.875 0 90)
 			(layer "F.SilkS")
 			(effects
@@
 		(tags "capacitor handsolder")
 		(property "Reference" "C1"
-			(at 0 -1.16 0)
+			(at -2.25 0.05 0)
 			(layer "F.SilkS")
 			(effects
@@
 		(tags "inductor handsolder")
 		(property "Reference" "L1"
-			(at 0 -1.17 0)
+			(at 1.925 0 0)
 			(layer "F.SilkS")
 			(effects
@@
 		(tags "test point SMD pad rectangle square")
 		(property "Reference" "TP2"
-			(at 0 -1.448 0)
+			(at 2.5 0.25 0)
 			(layer "F.SilkS")
 			(effects
@@
 		(tags "capacitor handsolder")
 		(property "Reference" "C3"
-			(at 0 -1.16 90)
+			(at 2.05 0 90)
 			(layer "F.SilkS")
 			(effects
@@
 		(tags "capacitor handsolder")
 		(property "Reference" "C2"
-			(at 0 -1.16 0)
+			(at 2.2 0 0)
 			(layer "F.SilkS")
 			(effects
@@
 		(tags "inductor handsolder")
 		(property "Reference" "FB7"
-			(at 0 -1.43 90)
+			(at -3.575 0 90)
 			(layer "F.SilkS")
 			(effects
@@
 		(tags "inductor handsolder")
 		(property "Reference" "L2"
-			(at 0 -1.17 90)
+			(at 2.075 -1.25 90)
 			(layer "F.SilkS")
 			(effects
@@
 		(tags "capacitor handsolder")
 		(property "Reference" "C25"
-			(at 0 -1.16 90)
+			(at 2.65 -0.05 90)
 			(layer "F.SilkS")
 			(effects
@@
 		(tags "capacitor handsolder")
 		(property "Reference" "C34"
-			(at 0 -1.16 90)
+			(at 2.45 -0.15 90)
 			(layer "F.SilkS")
 			(effects
@@
 		(at 145.5895 96.212)
 		(property "Reference" "U3"
-			(at -5.898 -13.494 0)
+			(at -10.5895 -9.012 0)
 			(layer "F.SilkS")
 			(effects
@@
 		(at 166.25 135.4127)
 		(property "Reference" "J3"
-			(at -0.325 -6.635 0)
+			(at 5.15 -1.4127 0)
 			(layer "F.SilkS")
 			(effects
@@
 		(tags "capacitor handsolder")
 		(property "Reference" "C29"
-			(at 0 -1.16 0)
+			(at 0 1.2 0)
 			(layer "F.SilkS")
 			(effects
@@
 		(tags "capacitor handsolder")
 		(property "Reference" "C32"
-			(at 0 -1.16 90)
+			(at 0 1.05 90)
 			(layer "F.SilkS")
 			(effects
@@
 		(layer "Edge.Cuts")
 	)
+	(gr_text "RF1"
+		(at 179.8 119.7 90)
+		(layer "F.SilkS")
+		(effects
+			(font
+				(size 1.5 1.5)
+				(thickness 0.2)
+			)
+			(justify left bottom)
+		)
+	)
+	(gr_text "RF2"
+		(at 157.4 134.6 0)
+		(layer "F.SilkS")
+		(effects
+			(font
+				(size 1.5 1.5)
+				(thickness 0.2)
+			)
+			(justify left bottom)
+		)
+	)
+	(gr_text "MX 2025"
+		(at 134.9 130.3 0)
+		(layer "F.SilkS")
+		(effects
+			(font
+				(size 1.5 1.5)
+				(thickness 0.2)
+			)
+			(justify left bottom)
+		)
+	)
+	(gr_text "LMX2594\nTest Board"
+		(at 179.7 103.2 90)
+		(layer "F.SilkS")
+		(effects
+			(font
+				(size 2 2)
+				(thickness 0.2)
+				(bold yes)
+			)
+			(justify left bottom)
+		)
+	)
 	(segment
 		(start 166.0675 114)
@@
 	)
 	(via
-		(at 133.7 87.2)
+		(at 134 88.1)
 		(size 0.6)
 		(drill 0.3)
@@
 	)
 	(via
-		(at 132 87.3)
-		(size 0.6)
-		(drill 0.3)
-		(layers "F.Cu" "B.Cu")
-		(free yes)
-		(net 1)
-	)
-	(via
-		(at 137.1 86)
-		(size 0.6)
-		(drill 0.3)
-		(layers "F.Cu" "B.Cu")
-		(free yes)
-		(net 1)
-	)
-	(via
 		(at 147.8 132.6)
 		(size 0.6)
@@
 	)
 	(via
-		(at 135.3 86)
-		(size 0.6)
-		(drill 0.3)
-		(layers "F.Cu" "B.Cu")
-		(free yes)
-		(net 1)
-	)
-	(via
 		(at 145.4 128.1)
 		(size 0.6)
@@
 	)
 	(via
-		(at 141.4 129.6)
+		(at 141.4 129.4)
 		(size 0.6)
 		(drill 0.3)
@@
 	)
 	(via
-		(at 136.7 130.3)
+		(at 136.8 130.6)
 		(size 0.6)
 		(drill 0.3)
@@
 	)
 	(via
-		(at 142.7 129.7)
+		(at 142.6 130.6)
 		(size 0.6)
 		(drill 0.3)
@@
 	)
 	(via
-		(at 136.7 128.6)
+		(at 136.8 129.3)
 		(size 0.6)
 		(drill 0.3)
@@
 	)
 	(via
-		(at 137.8 129.9)
+		(at 138.2 129.4)
 		(size 0.6)
 		(drill 0.3)
